Commit message: feat: prepare stir-fry grasp physics assets

File: isaac_assets/urdf/stirfry_bowl/stirfry_bowl.urdf (robot description, URDF)
Before this commit: robot stirfry_bowl, 1 links, 0 joints
Links:
- link base_link: geometry collision mesh filename=meshes/collision/bowl_collision_00_foot_high.stl scale=1 1 1; collision mesh filename=meshes/collision/bowl_collision_00_foot_low.stl scale=1 1 1
