Commit message: feat: update stir-fry tables to v2

File: isaac_assets/urdf/complete_table/complete_table.urdf (robot description, URDF)
Before this commit: robot complete_table, 1 links, 0 joints
Links:
- link base_link: mass 185.073375 -> 166.121232

File: isaac_assets/urdf/prepare_table/prepare_table.urdf (robot description, URDF)
Before this commit: robot prepare_table, 1 links, 0 joints
Links:
- link base_link: mass 263.845207 -> 226.232268

Commit message: fix: preserve stir-fry table bowl openings

File: isaac_assets/urdf/complete_table/complete_table.urdf (robot description, URDF)
Before this commit: robot complete_table, 1 links, 0 joints
Links:
- link base_link: geometry collision box size=0.045 0.045 0.810; collision box size=0.045 0.045 0.810

File: isaac_assets/urdf/prepare_table/prepare_table.urdf (robot description, URDF)
Before this commit: robot prepare_table, 1 links, 0 joints
Links:
- link base_link: geometry collision box size=0.025 1.099 0.075; collision box size=0.045 0.045 0.810
